Commit message: changed robots to turtlebot3

File: src/simulation/robot1/urdf/robot_description_urdf.urdf (robot description, URDF)
Before this commit: robot my_robot, 3 links, 2 joints
Links:
- removed link robot1_base_footprint
- added link base_footprint
- link base_link: geometry collision box size=0.3 0.3 0.1; visual box size=0.3 0.3 0.1
- link laser: geometry visual cylinder length=0.06 radius=0.04
Joints:
- joint base_joint: parent robot1_base_footprint -> base_footprint
- joint laser_joint: origin xyz=0 0 0.11 rpy=0 0 0 -> xyz=0 0 0.06 rpy=0 0 0
